File: HW/pocket_sdr_v2.1.brd (EAGLE design)
At the start: 55 x 21.6 mm, 75 parts, among them J1 PIN HEADER 2MM 2P, J2 PIN HEADER 2MM 2P, J3 USB MICRO B RECEPTACLE SMT, J4 SMA JACK EDGE MNT, U1 MAX2771, U2 MAX2771, U3 EZ-USB FX2LP CY7C6813A-56TXC, U4 AT24C128C 8-TSSOP, U5 LDO 3.3V 500mA SOT23-5

Commit message: TCXO 16.368 -> 24.000 MHz
Parts:
- TCXO: value 16.368 MHz -> 24.000 MHz
Changed lines of the file:
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@@
 <attribute name="NAME" x="28.1" y="17.2" size="0.8128" layer="25" font="vector" ratio="12"/>
 </element>
-<element name="TCXO" library="ttaka_misc" package="TCXO" value="16.368 MHz" x="25.1" y="16.55" smashed="yes" rot="R90">
+<element name="TCXO" library="ttaka_misc" package="TCXO" value="24.000 MHz" x="25.1" y="16.55" smashed="yes" rot="R90">
 <attribute name="NAME" x="25.495" y="15.264" size="0.8128" layer="21" font="vector" ratio="12" rot="R90"/>
 </element>
