File: HW/v2.3/pocket_sdr_v2.3.kicad_pcb (KiCad board)
At the start: 4 copper layers, 55 x 21.6 mm, 80 parts, among them J1 PINH_2MM_2P, J2 USB_C_Receptacle_USB2.0, J4 SMA-ANG, U1 MAX2771, U2 MAX2771, U3 CY7C68013A-56LTXCT, U4 AT24C128C, U5 LDO 3.3V 500mA SOT23-5

Commit message: Updated.
Parts:
- C36: value C1005 -> 100pF
Changed lines of the file:
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@@
         (effects (font (size 0.726968 0.726968) (thickness 0.085832)) (justify left bottom))
     )
-    (fp_text value "C1005" (at 0 0) (layer "F.Fab") hide
+    (fp_text value "100pF" (at 0 0) (layer "F.Fab") hide
         (effects (font (size 1.27 1.27) (thickness 0.15)))
     )
