File: HW/v2.3/pocket_sdr_v2.3.kicad_sch (KiCad schematic)
At the start: 76 parts, among them J1 PINH_2MM_2P, J2 USB_C_Receptacle_USB2.0, J4 SMA-ANG, U1 MAX2771, U2 MAX2771, U3 CY7C68013A-56LTXCT, U4 AT24C128C, U5 LDO 3.3V 500mA SOT23-5

Commit message: Updated.
Parts:
- C36: value C1005 -> 100pF
Changed lines of the file:
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@@
       (effects (font (size 1.27 1.0795)) (justify left bottom))
     )
-    (property "Value" "C1005" (at 50.165 276.225 0)
+    (property "Value" "100pF" (at 50.165 276.225 0)
       (effects (font (size 1.27 1.0795)) (justify left bottom))
     )
